Commit message: cleaned up some things

File: slam_bot/src/slambot_description/urdf/slambot.urdf (robot description, URDF)
Before this commit: robot slambot, 7 links, 6 joints
Links:
- removed link back_left_wheel
- removed link back_right_wheel
- removed link base_link
- removed link front_left_wheel
- removed link front_right_wheel
- removed link imu_link
- removed link laser_link
Joints:
- removed joint back_left_wheel_joint
- removed joint back_right_wheel_joint
- removed joint front_left_wheel_joint
- removed joint front_right_wheel_joint
- removed joint imu_mount
- removed joint laser_mount

File: slam_bot/src/slambot_description/urdf/slambot.xacro (robot description, xacro)
@@ -5,4 +5,6 @@
   <!-- If true in Gazebo Sim, move base kinematically from /cmd_vel (disables wheel physics effect) -->
   <xacro:arg name="kinematic" default="true"/>
+  <!-- Main robot macro so other files (e.g., .urdf wrapper) can include/instantiate -->
+  <xacro:macro name="slambot" params="">
   <!-- Base link with simple box visual and collision -->
   <link name="base_link">
@@ -295,5 +297,5 @@
           <twist_cov_diag>0.001 0.001 1000000 1000000 1000000 0.01</twist_cov_diag>
           <!-- Encoders (off by default to avoid conflicts) -->
-          <publish_encoders>false</publish_encoders>
+          <publish_encoders>true</publish_encoders>
           <ticks_topic>/wheel_ticks</ticks_topic>
           <joint_state_topic>/encoder_joint_states</joint_state_topic>
@@ -341,3 +343,6 @@
     </gazebo>
   </xacro:unless>
+  </xacro:macro>
+  <!-- Instantiate macro by default so this file remains directly usable with xacro -->
+  <xacro:slambot />
 </robot>
