Commit message: xacro file of the robot

File: slam_bot/src/slambot_description/urdf/slambot.xacro (robot description, xacro)
@@ -1,10 +1,16 @@
 <?xml version="1.0"?>
-<robot name="slambot">
+<robot xmlns:xacro="http://www.ros.org/wiki/xacro" name="slambot">
   <!-- Base link with simple box visual and collision -->
   <link name="base_link">
+    <inertial>
+      <!-- Raise base so its bottom touches wheel top (0.097 m) -->
+      <origin xyz="0 0 0.05" rpy="0 0 0"/>
+      <mass value="2.0"/>
+      <inertia ixx="0.011483" ixy="0.0" ixz="0.0" iyy="0.021483" iyz="0.0" izz="0.030833"/>
+    </inertial>
     <visual>
-      <origin xyz="0 0 0.04" rpy="0 0 0"/>
+      <origin xyz="0 0 0.05" rpy="0 0 0"/>
       <geometry>
-        <box size="0.35 0.25 0.08"/>
+        <box size="0.297 0.256 0.08"/>
       </geometry>
       <material name="gray">
@@ -13,7 +19,7 @@
     </visual>
     <collision>
-      <origin xyz="0 0 0.04" rpy="0 0 0"/>
+      <origin xyz="0 0 0.05" rpy="0 0 0"/>
       <geometry>
-        <box size="0.35 0.25 0.08"/>
+        <box size="0.297 0.256 0.08"/>
       </geometry>
     </collision>
@@ -21,6 +27,11 @@
   <!-- IMU -->
   <link name="imu_link">
+    <inertial>
+      <origin xyz="0 0 0.1" rpy="0 0 0"/>
+      <mass value="0.02"/>
+      <inertia ixx="3.333e-06" ixy="0.0" ixz="0.0" iyy="3.333e-06" iyz="0.0" izz="5.333e-06"/>
+    </inertial>
     <visual>
-      <origin xyz="0 0 0.10" rpy="0 0 0"/>
+      <origin xyz="0 0 0.1" rpy="0 0 0"/>
       <geometry>
         <box size="0.04 0.04 0.02"/>
@@ -31,5 +42,5 @@
     </visual>
     <collision>
-      <origin xyz="0 0 0.10" rpy="0 0 0"/>
+      <origin xyz="0 0 0.1" rpy="0 0 0"/>
       <geometry>
         <box size="0.04 0.04 0.02"/>
@@ -44,6 +55,11 @@
   <!-- LiDAR -->
   <link name="laser_link">
+    <inertial>
+      <origin xyz="0 0 -0.137" rpy="0 0 0"/>
+      <mass value="0.1"/>
+      <inertia ixx="4.396e-05" ixy="0.0" ixz="0.0" iyy="4.396e-05" iyz="0.0" izz="6.125e-05"/>
+    </inertial>
     <visual>
-      <origin xyz="0 0 0" rpy="0 0 0"/>
+      <origin xyz="0 0 -0.137" rpy="0 0 0"/>
       <geometry>
         <cylinder radius="0.035" length="0.04"/>
@@ -54,5 +70,5 @@
     </visual>
     <collision>
-      <origin xyz="0 0 0" rpy="0 0 0"/>
+      <origin xyz="0 0 -0.137" rpy="0 0 0"/>
       <geometry>
         <cylinder radius="0.035" length="0.04"/>
@@ -63,5 +79,5 @@
     <parent link="base_link"/>
     <child link="laser_link"/>
-    <origin xyz="0.10 0 0.15" rpy="0 0 0"/>
+    <origin xyz="0.10 0 0.247" rpy="0 0 0"/>
   </joint>
   <!-- Wheel parameters: radius=0.05m, width=0.02m
@@ -69,8 +85,13 @@
        Wheel cylinders are rotated so axis aligns with joint axis (y). -->
   <link name="front_left_wheel">
+    <inertial>
+      <origin xyz="0 0 0" rpy="1.5708 0 0"/>
+      <mass value="0.2"/>
+      <inertia ixx="0.0001317" ixy="0.0" ixz="0.0" iyy="0.00025" iyz="0.0" izz="0.0001317"/>
+    </inertial>
     <visual>
       <origin xyz="0 0 0" rpy="1.5708 0 0"/>
       <geometry>
-        <cylinder radius="0.05" length="0.02"/>
+        <cylinder radius="0.0485" length="0.048"/>
       </geometry>
       <material name="wheel_black">
@@ -81,5 +102,5 @@
       <origin xyz="0 0 0" rpy="1.5708 0 0"/>
       <geometry>
-        <cylinder radius="0.05" length="0.02"/>
+        <cylinder radius="0.0485" length="0.048"/>
       </geometry>
     </collision>
@@ -88,12 +109,17 @@
     <parent link="base_link"/>
     <child link="front_left_wheel"/>
-    <origin xyz="0.15 0.15 0.05" rpy="0 0 0"/>
+    <origin xyz="0.1485 0.152 0.0485" rpy="0 0 0"/>
     <axis xyz="0 1 0"/>
   </joint>
   <link name="front_right_wheel">
+    <inertial>
+      <origin xyz="0 0 0" rpy="1.5708 0 0"/>
+      <mass value="0.2"/>
+      <inertia ixx="0.0001317" ixy="0.0" ixz="0.0" iyy="0.00025" iyz="0.0" izz="0.0001317"/>
+    </inertial>
     <visual>
       <origin xyz="0 0 0" rpy="1.5708 0 0"/>
       <geometry>
-        <cylinder radius="0.05" length="0.02"/>
+        <cylinder radius="0.0485" length="0.048"/>
       </geometry>
       <material name="wheel_black"/>
@@ -102,5 +128,5 @@
       <origin xyz="0 0 0" rpy="1.5708 0 0"/>
       <geometry>
-        <cylinder radius="0.05" length="0.02"/>
+        <cylinder radius="0.0485" length="0.048"/>
       </geometry>
     </collision>
@@ -109,12 +135,17 @@
     <parent link="base_link"/>
     <child link="front_right_wheel"/>
-    <origin xyz="0.15 -0.15 0.05" rpy="0 0 0"/>
+    <origin xyz="0.1485 -0.152 0.0485" rpy="0 0 0"/>
     <axis xyz="0 1 0"/>
   </joint>
   <link name="back_left_wheel">
+    <inertial>
+      <origin xyz="0 0 0" rpy="1.5708 0 0"/>
+      <mass value="0.2"/>
+      <inertia ixx="0.0001317" ixy="0.0" ixz="0.0" iyy="0.00025" iyz="0.0" izz="0.0001317"/>
+    </inertial>
     <visual>
       <origin xyz="0 0 0" rpy="1.5708 0 0"/>
       <geometry>
-        <cylinder radius="0.05" length="0.02"/>
+        <cylinder radius="0.0485" length="0.048"/>
       </geometry>
       <material name="wheel_black"/>
@@ -123,5 +154,5 @@
       <origin xyz="0 0 0" rpy="1.5708 0 0"/>
       <geometry>
-        <cylinder radius="0.05" length="0.02"/>
+        <cylinder radius="0.0485" length="0.048"/>
       </geometry>
     </collision>
@@ -130,12 +161,17 @@
     <parent link="base_link"/>
     <child link="back_left_wheel"/>
-    <origin xyz="-0.15 0.15 0.05" rpy="0 0 0"/>
+    <origin xyz="-0.1485 0.152 0.0485" rpy="0 0 0"/>
     <axis xyz="0 1 0"/>
   </joint>
   <link name="back_right_wheel">
+    <inertial>
+      <origin xyz="0 0 0" rpy="1.5708 0 0"/>
+      <mass value="0.2"/>
+      <inertia ixx="0.0001317" ixy="0.0" ixz="0.0" iyy="0.00025" iyz="0.0" izz="0.0001317"/>
+    </inertial>
     <visual>
       <origin xyz="0 0 0" rpy="1.5708 0 0"/>
       <geometry>
-        <cylinder radius="0.05" length="0.02"/>
+        <cylinder radius="0.0485" length="0.048"/>
       </geometry>
       <material name="wheel_black"/>
@@ -144,5 +180,5 @@
       <origin xyz="0 0 0" rpy="1.5708 0 0"/>
       <geometry>
-        <cylinder radius="0.05" length="0.02"/>
+        <cylinder radius="0.0485" length="0.048"/>
       </geometry>
     </collision>
@@ -151,5 +187,5 @@
     <parent link="base_link"/>
     <child link="back_right_wheel"/>
-    <origin xyz="-0.15 -0.15 0.05" rpy="0 0 0"/>
+    <origin xyz="-0.1485 -0.152 0.0485" rpy="0 0 0"/>
     <axis xyz="0 1 0"/>
   </joint>

Commit message: added mecanum drive in sim

File: slam_bot/src/slambot_description/urdf/slambot.xacro (robot description, xacro)
@@ -1,4 +1,6 @@
 <?xml version="1.0"?>
 <robot xmlns:xacro="http://www.ros.org/wiki/xacro" name="slambot">
+  <!-- Simulation flavor: true = Gazebo Sim (Ignition) via gz_ros2_control, false = Gazebo Classic -->
+  <xacro:arg name="use_gz" default="true"/>
   <!-- Base link with simple box visual and collision -->
   <link name="base_link">
@@ -190,3 +192,126 @@
     <axis xyz="0 1 0"/>
   </joint>
+  <transmission name="front_left_transmission">
+    <type>transmission_interface/SimpleTransmission</type>
+    <joint name="front_left_wheel_joint">
+      <hardwareInterface>hardware_interface/VelocityCommandInterface</hardwareInterface>
+    </joint>
+    <actuator name="front_left_motor">
+      <hardwareInterface>hardware_interface/VelocityCommandInterface</hardwareInterface>
+      <mechanicalReduction>1</mechanicalReduction>
+    </actuator>
+  </transmission>
+  <transmission name="front_right_transmission">
+    <type>transmission_interface/SimpleTransmission</type>
+    <joint name="front_right_wheel_joint">
+      <hardwareInterface>hardware_interface/VelocityCommandInterface</hardwareInterface>
+    </joint>
+    <actuator name="front_right_motor">
+      <hardwareInterface>hardware_interface/VelocityCommandInterface</hardwareInterface>
+      <mechanicalReduction>1</mechanicalReduction>
+    </actuator>
+  </transmission>
+  <transmission name="back_left_transmission">
+    <type>transmission_interface/SimpleTransmission</type>
+    <joint name="back_left_wheel_joint">
+      <hardwareInterface>hardware_interface/VelocityCommandInterface</hardwareInterface>
+    </joint>
+    <actuator name="back_left_motor">
+      <hardwareInterface>hardware_interface/VelocityCommandInterface</hardwareInterface>
+      <mechanicalReduction>1</mechanicalReduction>
+    </actuator>
+  </transmission>
+  <transmission name="back_right_transmission">
+    <type>transmission_interface/SimpleTransmission</type>
+    <joint name="back_right_wheel_joint">
+      <hardwareInterface>hardware_interface/VelocityCommandInterface</hardwareInterface>
+    </joint>
+    <actuator name="back_right_motor">
+      <hardwareInterface>hardware_interface/VelocityCommandInterface</hardwareInterface>
+      <mechanicalReduction>1</mechanicalReduction>
+    </actuator>
+  </transmission>
+  <!-- ros2_control interfaces; hardware plugin varies by sim flavor -->
+  <ros2_control name="slambot_system" type="system">
+    <xacro:if value="$(arg use_gz)">
+      <hardware>
+        <plugin>gz_ros2_control/GazeboSimSystem</plugin>
+      </hardware>
+    </xacro:if>
+    <xacro:unless value="$(arg use_gz)">
+      <hardware>
+        <plugin>gazebo_ros2_control/GazeboSystem</plugin>
+      </hardware>
+    </xacro:unless>
+    <joint name="front_left_wheel_joint">
+      <command_interface name="velocity"/>
+      <state_interface name="position"/>
+      <state_interface name="velocity"/>
+    </joint>
+    <joint name="front_right_wheel_joint">
+      <command_interface name="velocity"/>
+      <state_interface name="position"/>
+      <state_interface name="velocity"/>
+    </joint>
+    <joint name="back_left_wheel_joint">
+      <command_interface name="velocity"/>
+      <state_interface name="position"/>
+      <state_interface name="velocity"/>
+    </joint>
+    <joint name="back_right_wheel_joint">
+      <command_interface name="velocity"/>
+      <state_interface name="position"/>
+      <state_interface name="velocity"/>
+    </joint>
+  </ros2_control>
+  <xacro:if value="$(arg use_gz)">
+    <gazebo>
+      <plugin
+          name="gz_ros2_control::GazeboSimROS2ControlPlugin"
+          filename="libgz_ros2_control-system.so">
+        <ros2_control>
+          slambot_system
+        </ros2_control>
+        <!-- Path to controller manager parameters YAML -->
+        <parameters>$(find slambot_description)/config/mecanum_controller.yaml</parameters>
+      </plugin>
+      <!-- Kinematic base controller: apply /cmd_vel directly to model velocity (Gazebo Sim) -->
+      <plugin name="slambot_kinematic_base" filename="libslambot_kinematic_base.so">
+        <topic>/cmd_vel</topic>
+        <max_linear>1.5</max_linear>
+        <max_angular>3.0</max_angular>
+      </plugin>
+    </gazebo>
+  </xacro:if>
+  <xacro:unless value="$(arg use_gz)">
+    <gazebo>
+      <plugin name="gazebo_ros2_control" filename="libgazebo_ros2_control.so">
+        <!-- Path to controller manager parameters YAML -->
+        <parameters>$(find slambot_description)/config/mecanum_controller.yaml</parameters>
+      </plugin>
+    </gazebo>
+  </xacro:unless>
+  <!-- Approximate mecanum behavior via anisotropic friction directions (Gazebo Classic ODE only) -->
+  <xacro:unless value="$(arg use_gz)">
+    <gazebo reference="front_left_wheel">
+      <mu1>1.0</mu1>
+      <mu2>0.05</mu2>
+      <fdir1>1 1 0</fdir1>
+    </gazebo>
+    <gazebo reference="front_right_wheel">
+      <mu1>1.0</mu1>
+      <mu2>0.05</mu2>
+      <fdir1>1 -1 0</fdir1>
+    </gazebo>
+    <gazebo reference="back_left_wheel">
+      <mu1>1.0</mu1>
+      <mu2>0.05</mu2>
+      <fdir1>-1 -1 0</fdir1>
+    </gazebo>
+    <gazebo reference="back_right_wheel">
+      <mu1>1.0</mu1>
+      <mu2>0.05</mu2>
+      <fdir1>-1 1 0</fdir1>
+    </gazebo>
+  </xacro:unless>
 </robot>

Commit message: better rotation odom

File: slam_bot/src/slambot_description/urdf/slambot.xacro (robot description, xacro)
@@ -7,4 +7,10 @@
   <!-- Main robot macro so other files (e.g., .urdf wrapper) can include/instantiate -->
   <xacro:macro name="slambot" params="">
+  <xacro:property name="robot_length" value="0.297"/>  <!-- m -->
+  <xacro:property name="robot_width" value="0.256"/>   <!-- m -->
+  <xacro:property name="wheel_radius" value="0.0485"/>   <!-- m -->
+  <xacro:property name="robot_height" value="0.08"/>    <!-- m -->
+  <xacro:property name="battery_depth" value="0.051"/>  <!-- m, 2 inches out -->
+  <xacro:property name="battery_width" value="0.281"/>  <!-- m, robot_width + 1 inch (0.5in on each side) -->
   <!-- Base link with simple box visual and collision -->
   <link name="base_link">
@@ -18,5 +24,5 @@
       <origin xyz="0 0 0.05" rpy="0 0 0"/>
       <geometry>
-        <box size="0.297 0.256 0.08"/>
+        <box size="${robot_length} ${robot_width} ${robot_height}"/>
       </geometry>
       <material name="gray">
@@ -27,8 +33,36 @@
       <origin xyz="0 0 0.05" rpy="0 0 0"/>
       <geometry>
-        <box size="0.297 0.256 0.08"/>
-      </geometry>
-    </collision>
-  </link>
+        <box size="${robot_length} ${robot_width} ${robot_height}"/>
+      </geometry>
+    </collision>
+  </link>
+  <!-- Battery Pack -->
+  <link name="battery_link">
+    <inertial>
+      <origin xyz="0 0 0.06" rpy="0 0 0"/>
+      <mass value="0.5"/>
+      <inertia ixx="0.000417" ixy="0.0" ixz="0.0" iyy="0.000417" iyz="0.0" izz="0.000278"/>
+    </inertial>
+    <visual>
+      <origin xyz="0 0 0.06" rpy="0 0 0"/>
+      <geometry>
+        <box size="${battery_depth} ${battery_width} 0.04"/>
+      </geometry>
+      <material name="red">
+        <color rgba="0.9 0.1 0.1 1.0"/>
+      </material>
+    </visual>
+    <collision>
+      <origin xyz="0 0 0.06" rpy="0 0 0"/>
+      <geometry>
+        <box size="${battery_depth} ${battery_width} 0.04"/>
+      </geometry>
+    </collision>
+  </link>
+  <joint name="battery_mount" type="fixed">
+    <parent link="base_link"/>
+    <child link="battery_link"/>
+    <origin xyz="-0.174 0 0" rpy="0 0 0"/>
+  </joint>
   <!-- IMU -->
   <link name="imu_link">
@@ -41,5 +75,5 @@
       <origin xyz="0 0 0.1" rpy="0 0 0"/>
       <geometry>
-        <box size="0.04 0.04 0.02"/>
+        <box size="0.02 0.02 0.01"/>
       </geometry>
       <material name="blue">
@@ -50,5 +84,5 @@
       <origin xyz="0 0 0.1" rpy="0 0 0"/>
       <geometry>
-        <box size="0.04 0.04 0.02"/>
+        <box size="0.02 0.02 0.01"/>
       </geometry>
     </collision>
@@ -57,5 +91,5 @@
     <parent link="base_link"/>
     <child link="imu_link"/>
-    <origin xyz="0 0 0" rpy="0 0 3.1415926535"/>
+    <origin xyz="-0.048 0 0" rpy="0 0 3.1415926535"/>
   </joint>
   <!-- LiDAR -->
@@ -87,6 +121,6 @@
     <origin xyz="0.10 0 0.247" rpy="0 0 0"/>
   </joint>
-  <!-- Wheel parameters: radius=0.05m, width=0.02m
-       Track width (y): +/-0.15m, Wheelbase (x): +/-0.15m
+  <!-- Wheel parameters: radius=0.0485m, width=0.048m
+       Track width (y): +/-0.152m, Wheelbase (x): +/-0.097m (0.194m total, 7.625 inches)
        Wheel cylinders are rotated so axis aligns with joint axis (y). -->
   <link name="front_left_wheel">
@@ -99,5 +133,5 @@
       <origin xyz="0 0 0" rpy="1.5708 0 0"/>
       <geometry>
-        <cylinder radius="0.0485" length="0.048"/>
+        <cylinder radius="${wheel_radius}" length="0.048"/>
       </geometry>
       <material name="wheel_black">
@@ -108,5 +142,5 @@
       <origin xyz="0 0 0" rpy="1.5708 0 0"/>
       <geometry>
-        <cylinder radius="0.0485" length="0.048"/>
+        <cylinder radius="${wheel_radius}" length="0.048"/>
       </geometry>
     </collision>
@@ -115,5 +149,5 @@
     <parent link="base_link"/>
     <child link="front_left_wheel"/>
-    <origin xyz="0.1485 0.152 0.0485" rpy="0 0 0"/>
+    <origin xyz="0.097 0.152 ${wheel_radius}" rpy="0 0 0"/>
     <axis xyz="0 1 0"/>
   </joint>
@@ -127,5 +161,5 @@
       <origin xyz="0 0 0" rpy="1.5708 0 0"/>
       <geometry>
-        <cylinder radius="0.0485" length="0.048"/>
+        <cylinder radius="${wheel_radius}" length="0.048"/>
       </geometry>
       <material name="wheel_black"/>
@@ -134,5 +168,5 @@
       <origin xyz="0 0 0" rpy="1.5708 0 0"/>
       <geometry>
-        <cylinder radius="0.0485" length="0.048"/>
+        <cylinder radius="${wheel_radius}" length="0.048"/>
       </geometry>
     </collision>
@@ -141,5 +175,5 @@
     <parent link="base_link"/>
     <child link="front_right_wheel"/>
-    <origin xyz="0.1485 -0.152 0.0485" rpy="0 0 0"/>
+    <origin xyz="0.097 -0.152 ${wheel_radius}" rpy="0 0 0"/>
     <axis xyz="0 1 0"/>
   </joint>
@@ -153,5 +187,5 @@
       <origin xyz="0 0 0" rpy="1.5708 0 0"/>
       <geometry>
-        <cylinder radius="0.0485" length="0.048"/>
+        <cylinder radius="${wheel_radius}" length="0.048"/>
       </geometry>
       <material name="wheel_black"/>
@@ -160,5 +194,5 @@
       <origin xyz="0 0 0" rpy="1.5708 0 0"/>
       <geometry>
-        <cylinder radius="0.0485" length="0.048"/>
+        <cylinder radius="${wheel_radius}" length="0.048"/>
       </geometry>
     </collision>
@@ -167,5 +201,5 @@
     <parent link="base_link"/>
     <child link="back_left_wheel"/>
-    <origin xyz="-0.1485 0.152 0.0485" rpy="0 0 0"/>
+    <origin xyz="-0.097 0.152 ${wheel_radius}" rpy="0 0 0"/>
     <axis xyz="0 1 0"/>
   </joint>
@@ -179,5 +213,5 @@
       <origin xyz="0 0 0" rpy="1.5708 0 0"/>
       <geometry>
-        <cylinder radius="0.0485" length="0.048"/>
+        <cylinder radius="${wheel_radius}" length="0.048"/>
       </geometry>
       <material name="wheel_black"/>
@@ -186,5 +220,5 @@
       <origin xyz="0 0 0" rpy="1.5708 0 0"/>
       <geometry>
-        <cylinder radius="0.0485" length="0.048"/>
+        <cylinder radius="${wheel_radius}" length="0.048"/>
       </geometry>
     </collision>
@@ -193,5 +227,5 @@
     <parent link="base_link"/>
     <child link="back_right_wheel"/>
-    <origin xyz="-0.1485 -0.152 0.0485" rpy="0 0 0"/>
+    <origin xyz="-0.097 -0.152 ${wheel_radius}" rpy="0 0 0"/>
     <axis xyz="0 1 0"/>
   </joint>
@@ -298,10 +332,12 @@
           <!-- Encoders (off by default to avoid conflicts) -->
           <publish_encoders>true</publish_encoders>
-          <ticks_topic>/wheel_ticks</ticks_topic>
+          <ticks_topic>/wheel_encoders</ticks_topic>
           <joint_state_topic>/encoder_joint_states</joint_state_topic>
-          <ticks_per_rev>2048</ticks_per_rev>
-          <wheel_radius>0.0485</wheel_radius>
-          <base_length>0.297</base_length>
-          <base_width>0.256</base_width>
+          <ticks_per_rev>2880</ticks_per_rev>
+          <wheel_radius>${wheel_radius}</wheel_radius>
+          <!-- base_length and base_width for mecanum kinematics must be wheel-to-wheel distances, NOT robot dimensions -->
+          <!-- Measured: 210mm length (front-to-back), 195mm width (left-to-right) -->
+          <base_length>0.21</base_length>
+          <base_width>0.1925</base_width>
           <front_left_joint>front_left_wheel_joint</front_left_joint>
           <front_right_joint>front_right_wheel_joint</front_right_joint>
