Commit message: cleaned up xacro and added imu to sim, sim is now as similar to real life as possible

File: slam_bot/src/slambot_description/urdf/slambot.xacro (robot description, xacro)
@@ -7,27 +7,6 @@
   <!-- Main robot macro so other files (e.g., .urdf wrapper) can include/instantiate -->
   <xacro:macro name="slambot" params="">
-    <!-- =========================
-         VISUAL / BODY DIMENSIONS
-         (These are "what it looks like")
-         ========================= -->
-    <xacro:property name="robot_length" value="0.297"/>  <!-- m (overall body box you chose) -->
-    <xacro:property name="robot_width"  value="0.152"/>  <!-- m (overall width you chose) -->
-    <xacro:property name="robot_height" value="0.08"/>   <!-- m -->
-    <!-- Wheel geometry -->
-    <xacro:property name="wheel_radius" value="0.0485"/> <!-- m -->
-    <xacro:property name="wheel_thickness" value="0.048"/> <!-- m (cylinder length) -->
-    <!-- =========================
-         REAL-LIFE WHEEL-CENTER GEOMETRY
-         (This is what controls motion accuracy)
-         These MUST match what worked IRL.
-         ========================= -->
-    <xacro:property name="base_length" value="0.21"/>  <!-- m: wheel center-to-center front↔back -->
-    <xacro:property name="base_width"  value="0.200"/> <!-- m: wheel center-to-center left↔right -->
-    <!-- Convenience: half distances -->
-    <xacro:property name="wheel_x" value="${base_length/2.0}"/>
-    <xacro:property name="wheel_y" value="${base_width/2.0}"/>
-    <!-- Battery -->
-    <xacro:property name="battery_depth" value="0.051"/>  <!-- m -->
-    <xacro:property name="battery_width" value="0.177"/>  <!-- m -->
+    <!-- Parameters -->
+    <xacro:include filename="$(find slambot_description)/urdf/slambot-params.xacro" />
     <!-- Base link with simple box visual and collision -->
     <link name="base_link">
@@ -81,212 +60,13 @@
       <origin xyz="-0.174 0 0" rpy="0 0 0"/>
     </joint>
-    <!-- IMU -->
-    <link name="imu_link">
-      <inertial>
-        <origin xyz="0 0 0.1" rpy="0 0 0"/>
-        <mass value="0.02"/>
-        <inertia ixx="3.333e-06" ixy="0.0" ixz="0.0" iyy="3.333e-06" iyz="0.0" izz="5.333e-06"/>
-      </inertial>
-      <visual>
-        <origin xyz="0 0 0.1" rpy="0 0 0"/>
-        <geometry>
-          <box size="0.02 0.02 0.01"/>
-        </geometry>
-        <material name="blue">
-          <color rgba="0.2 0.4 0.9 1.0"/>
-        </material>
-      </visual>
-      <collision>
-        <origin xyz="0 0 0.1" rpy="0 0 0"/>
-        <geometry>
-          <box size="0.02 0.02 0.01"/>
-        </geometry>
-      </collision>
-    </link>
-    <joint name="imu_mount" type="fixed">
-      <parent link="base_link"/>
-      <child link="imu_link"/>
-      <origin xyz="-0.048 0 0" rpy="0 0 3.1415926535"/>
-    </joint>
-    <!-- LiDAR -->
-    <link name="laser_link">
-      <inertial>
-        <origin xyz="0 0 -0.137" rpy="0 0 0"/>
-        <mass value="0.1"/>
-        <inertia ixx="4.396e-05" ixy="0.0" ixz="0.0" iyy="4.396e-05" iyz="0.0" izz="6.125e-05"/>
-      </inertial>
-      <visual>
-        <origin xyz="0 0 -0.137" rpy="0 0 0"/>
-        <geometry>
-          <cylinder radius="0.035" length="0.04"/>
-        </geometry>
-        <material name="black">
-          <color rgba="0.1 0.1 0.1 1.0"/>
-        </material>
-      </visual>
-      <collision>
-        <origin xyz="0 0 -0.137" rpy="0 0 0"/>
-        <geometry>
-          <cylinder radius="0.035" length="0.04"/>
-        </geometry>
-      </collision>
-    </link>
-    <joint name="laser_mount" type="fixed">
-      <parent link="base_link"/>
-      <child link="laser_link"/>
-      <origin xyz="0.10 0 0.247" rpy="0 0 0"/>
-    </joint>
-    <!-- =========================
-         WHEELS (UPDATED POSITIONS)
-         wheel_x = base_length/2
-         wheel_y = base_width/2
-         ========================= -->
-    <link name="front_left_wheel">
-      <inertial>
-        <origin xyz="0 0 0" rpy="1.5708 0 0"/>
-        <mass value="0.2"/>
-        <inertia ixx="0.0001317" ixy="0.0" ixz="0.0" iyy="0.00025" iyz="0.0" izz="0.0001317"/>
-      </inertial>
-      <visual>
-        <origin xyz="0 0 0" rpy="1.5708 0 0"/>
-        <geometry>
-          <cylinder radius="${wheel_radius}" length="${wheel_thickness}"/>
-        </geometry>
-        <material name="wheel_black">
-          <color rgba="0.05 0.05 0.05 1.0"/>
-        </material>
-      </visual>
-      <collision>
-        <origin xyz="0 0 0" rpy="1.5708 0 0"/>
-        <geometry>
-          <cylinder radius="${wheel_radius}" length="${wheel_thickness}"/>
-        </geometry>
-      </collision>
-    </link>
-    <joint name="front_left_wheel_joint" type="continuous">
-      <parent link="base_link"/>
-      <child link="front_left_wheel"/>
-      <origin xyz="${wheel_x} ${wheel_y} ${wheel_radius}" rpy="0 0 0"/>
-      <axis xyz="0 1 0"/>
-    </joint>
-    <link name="front_right_wheel">
-      <inertial>
-        <origin xyz="0 0 0" rpy="1.5708 0 0"/>
-        <mass value="0.2"/>
-        <inertia ixx="0.0001317" ixy="0.0" ixz="0.0" iyy="0.00025" iyz="0.0" izz="0.0001317"/>
-      </inertial>
-      <visual>
-        <origin xyz="0 0 0" rpy="1.5708 0 0"/>
-        <geometry>
-          <cylinder radius="${wheel_radius}" length="${wheel_thickness}"/>
-        </geometry>
-        <material name="wheel_black"/>
-      </visual>
-      <collision>
-        <origin xyz="0 0 0" rpy="1.5708 0 0"/>
-        <geometry>
-          <cylinder radius="${wheel_radius}" length="${wheel_thickness}"/>
-        </geometry>
-      </collision>
-    </link>
-    <joint name="front_right_wheel_joint" type="continuous">
-      <parent link="base_link"/>
-      <child link="front_right_wheel"/>
-      <origin xyz="${wheel_x} ${-wheel_y} ${wheel_radius}" rpy="0 0 0"/>
-      <axis xyz="0 1 0"/>
-    </joint>
-    <link name="back_left_wheel">
-      <inertial>
-        <origin xyz="0 0 0" rpy="1.5708 0 0"/>
-        <mass value="0.2"/>
-        <inertia ixx="0.0001317" ixy="0.0" ixz="0.0" iyy="0.00025" iyz="0.0" izz="0.0001317"/>
-      </inertial>
-      <visual>
-        <origin xyz="0 0 0" rpy="1.5708 0 0"/>
-        <geometry>
-          <cylinder radius="${wheel_radius}" length="${wheel_thickness}"/>
-        </geometry>
-        <material name="wheel_black"/>
-      </visual>
-      <collision>
-        <origin xyz="0 0 0" rpy="1.5708 0 0"/>
-        <geometry>
-          <cylinder radius="${wheel_radius}" length="${wheel_thickness}"/>
-        </geometry>
-      </collision>
-    </link>
-    <joint name="back_left_wheel_joint" type="continuous">
-      <parent link="base_link"/>
-      <child link="back_left_wheel"/>
-      <origin xyz="${-wheel_x} ${wheel_y} ${wheel_radius}" rpy="0 0 0"/>
-      <axis xyz="0 1 0"/>
-    </joint>
-    <link name="back_right_wheel">
-      <inertial>
-        <origin xyz="0 0 0" rpy="1.5708 0 0"/>
-        <mass value="0.2"/>
-        <inertia ixx="0.0001317" ixy="0.0" ixz="0.0" iyy="0.00025" iyz="0.0" izz="0.0001317"/>
-      </inertial>
-      <visual>
-        <origin xyz="0 0 0" rpy="1.5708 0 0"/>
-        <geometry>
-          <cylinder radius="${wheel_radius}" length="${wheel_thickness}"/>
-        </geometry>
-        <material name="wheel_black"/>
-      </visual>
-      <collision>
-        <origin xyz="0 0 0" rpy="1.5708 0 0"/>
-        <geometry>
-          <cylinder radius="${wheel_radius}" length="${wheel_thickness}"/>
-        </geometry>
-      </collision>
-    </link>
-    <joint name="back_right_wheel_joint" type="continuous">
-      <parent link="base_link"/>
-      <child link="back_right_wheel"/>
-      <origin xyz="${-wheel_x} ${-wheel_y} ${wheel_radius}" rpy="0 0 0"/>
-      <axis xyz="0 1 0"/>
-    </joint>
-    <!-- Transmissions (unchanged) -->
-    <transmission name="front_left_transmission">
-      <type>transmission_interface/SimpleTransmission</type>
-      <joint name="front_left_wheel_joint">
-        <hardwareInterface>hardware_interface/VelocityCommandInterface</hardwareInterface>
-      </joint>
-      <actuator name="front_left_motor">
-        <hardwareInterface>hardware_interface/VelocityCommandInterface</hardwareInterface>
-        <mechanicalReduction>1</mechanicalReduction>
-      </actuator>
-    </transmission>
-    <transmission name="front_right_transmission">
-      <type>transmission_interface/SimpleTransmission</type>
-      <joint name="front_right_wheel_joint">
-        <hardwareInterface>hardware_interface/VelocityCommandInterface</hardwareInterface>
-      </joint>
-      <actuator name="front_right_motor">
-        <hardwareInterface>hardware_interface/VelocityCommandInterface</hardwareInterface>
-        <mechanicalReduction>1</mechanicalReduction>
-      </actuator>
-    </transmission>
-    <transmission name="back_left_transmission">
-      <type>transmission_interface/SimpleTransmission</type>
-      <joint name="back_left_wheel_joint">
-        <hardwareInterface>hardware_interface/VelocityCommandInterface</hardwareInterface>
-      </joint>
-      <actuator name="back_left_motor">
-        <hardwareInterface>hardware_interface/VelocityCommandInterface</hardwareInterface>
-        <mechanicalReduction>1</mechanicalReduction>
-      </actuator>
-    </transmission>
-    <transmission name="back_right_transmission">
-      <type>transmission_interface/SimpleTransmission</type>
-      <joint name="back_right_wheel_joint">
-        <hardwareInterface>hardware_interface/VelocityCommandInterface</hardwareInterface>
-      </joint>
-      <actuator name="back_right_motor">
-        <hardwareInterface>hardware_interface/VelocityCommandInterface</hardwareInterface>
-        <mechanicalReduction>1</mechanicalReduction>
-      </actuator>
-    </transmission>
+    <!-- Sensors (IMU) split out for clarity -->
+    <xacro:include filename="$(find slambot_description)/urdf/slambot-sensors.xacro" />
+    <xacro:slambot_imu />
+    <!-- Wheels split out for clarity -->
+    <xacro:include filename="$(find slambot_description)/urdf/slambot-wheels.xacro" />
+    <xacro:slambot_wheels />
+    <!-- Transmissions split out for clarity -->
+    <xacro:include filename="$(find slambot_description)/urdf/slambot-transmissions.xacro" />
+    <xacro:slambot_transmissions />
     <!-- ros2_control interfaces; hardware plugin varies by sim flavor -->
     <ros2_control name="slambot_system" type="system">
@@ -347,5 +127,5 @@
             <ticks_topic>/wheel_encoders</ticks_topic>
             <joint_state_topic>/encoder_joint_states</joint_state_topic>
-            <ticks_per_rev>2880</ticks_per_rev>
+            <ticks_per_rev>2882</ticks_per_rev>
             <wheel_radius>${wheel_radius}</wheel_radius>
             <!-- IMPORTANT: These now match your IRL tuned values -->
@@ -367,27 +147,4 @@
       </gazebo>
     </xacro:unless>
-    <!-- Approximate mecanum behavior via anisotropic friction directions (Gazebo Classic ODE only) -->
-    <xacro:unless value="$(arg use_gz)">
-      <gazebo reference="front_left_wheel">
-        <mu1>1.0</mu1>
-        <mu2>0.05</mu2>
-        <fdir1>1 1 0</fdir1>
-      </gazebo>
-      <gazebo reference="front_right_wheel">
-        <mu1>1.0</mu1>
-        <mu2>0.05</mu2>
-        <fdir1>1 -1 0</fdir1>
-      </gazebo>
-      <gazebo reference="back_left_wheel">
-        <mu1>1.0</mu1>
-        <mu2>0.05</mu2>
-        <fdir1>-1 -1 0</fdir1>
-      </gazebo>
-      <gazebo reference="back_right_wheel">
-        <mu1>1.0</mu1>
-        <mu2>0.05</mu2>
-        <fdir1>-1 1 0</fdir1>
-      </gazebo>
-    </xacro:unless>
   </xacro:macro>
   <!-- Instantiate macro by default so this file remains directly usable with xacro -->
