Commit message: got rid of unused ros2 control and added lidar to sim

File: slam_bot/src/slambot_description/urdf/slambot-sensors.xacro (robot description, xacro)
@@ -76,4 +76,178 @@
       </gazebo>
     </xacro:if>
+    <!--
+      LIDAR platform and GPU lidar mounted above the IMU.
+      - Four visual pegs/standoffs lift a small plate ~2 inches (0.0508 m) above the IMU frame.
+      - A lidar link is mounted on the plate and equipped with a GPU lidar sensor.
+    -->
+    <!-- Lidar mounting plate, positioned above the IMU -->
+    <link name="lidar_plate_link">
+      <inertial>
+        <origin xyz="0 0 0" rpy="0 0 0"/>
+        <mass value="0.05"/>
+        <inertia ixx="1e-4" ixy="0" ixz="0" iyy="1e-4" iyz="0" izz="1e-4"/>
+      </inertial>
+      <!-- Thin plate -->
+      <visual>
+        <origin xyz="0 0 0" rpy="0 0 0"/>
+        <geometry>
+          <box size="0.10 0.10 0.003"/>
+        </geometry>
+        <material name="dark_gray">
+          <color rgba="0.3 0.3 0.3 1.0"/>
+        </material>
+      </visual>
+      <collision>
+        <origin xyz="0 0 0" rpy="0 0 0"/>
+        <geometry>
+          <box size="0.10 0.10 0.003"/>
+        </geometry>
+      </collision>
+      <!-- Four standoffs/pegs (visual only) placed at the corners, extending down to chassis top -->
+      <visual>
+        <!-- L = 0.0658, origin.z = -0.0344 so top meets plate underside, bottom meets chassis top -->
+        <origin xyz=" 0.045  0.045 -0.0344" rpy="0 0 0"/>
+        <geometry>
+          <cylinder radius="0.004" length="0.0658"/>
+        </geometry>
+        <material name="black">
+          <color rgba="0.1 0.1 0.1 1.0"/>
+        </material>
+      </visual>
+      <visual>
+        <origin xyz=" 0.045 -0.045 -0.0344" rpy="0 0 0"/>
+        <geometry>
+          <cylinder radius="0.004" length="0.0658"/>
+        </geometry>
+        <material name="black"/>
+      </visual>
+      <visual>
+        <origin xyz="-0.045  0.045 -0.0344" rpy="0 0 0"/>
+        <geometry>
+          <cylinder radius="0.004" length="0.0658"/>
+        </geometry>
+        <material name="black"/>
+      </visual>
+      <visual>
+        <origin xyz="-0.045 -0.045 -0.0344" rpy="0 0 0"/>
+        <geometry>
+          <cylinder radius="0.004" length="0.0658"/>
+        </geometry>
+        <material name="black"/>
+      </visual>
+    </link>
+    <joint name="lidar_plate_joint" type="fixed">
+      <parent link="base_link"/>
+      <!-- Place plate ~2 in above IMU top; pegs rest on chassis top.
+           base top z=0.09, imu top z≈0.105 → plate underside ≈ 0.105+0.0508=0.1558
+           plate center = underside + 0.0015 = 0.1573 -->
+      <child link="lidar_plate_link"/>
+      <origin xyz="0 0 0.1573" rpy="0 0 0"/>
+    </joint>
+    <!-- Lidar body/link mounted on top of the plate -->
+    <link name="gpu_lidar_link">
+      <inertial>
+        <origin xyz="0 0 0" rpy="0 0 0"/>
+        <mass value="0.15"/>
+        <inertia ixx="2e-4" ixy="0" ixz="0" iyy="2e-4" iyz="0" izz="2e-4"/>
+      </inertial>
+      <visual>
+        <!-- Small puck-style lidar -->
+        <origin xyz="0 0 0" rpy="0 0 0"/>
+        <geometry>
+          <cylinder radius="0.035" length="0.025"/>
+        </geometry>
+        <material name="blue">
+          <color rgba="0.2 0.4 0.9 1.0"/>
+        </material>
+      </visual>
+      <collision>
+        <origin xyz="0 0 0" rpy="0 0 0"/>
+        <geometry>
+          <cylinder radius="0.035" length="0.025"/>
+        </geometry>
+      </collision>
+    </link>
+    <joint name="gpu_lidar_mount" type="fixed">
+      <parent link="lidar_plate_link"/>
+      <child link="gpu_lidar_link"/>
+      <!-- Sit the lidar on plate top: z = plate half-thickness + lidar half-length = 0.0015 + 0.0125 -->
+      <origin xyz="0 0 0.014" rpy="0 0 0"/>
+    </joint>
+    <!-- Gazebo Classic GPU lidar (only when NOT using Gazebo Sim) -->
+    <xacro:unless value="$(arg use_gz)">
+      <gazebo reference="gpu_lidar_link">
+        <sensor name="gpu_lidar" type="gpu_ray">
+          <always_on>1</always_on>
+          <update_rate>20</update_rate>
+          <visualize>true</visualize>
+          <ray>
+            <scan>
+              <horizontal>
+                <samples>720</samples>
+                <resolution>1</resolution>
+                <min_angle>-3.14159</min_angle>
+                <max_angle>3.14159</max_angle>
+              </horizontal>
+              <vertical>
+                <samples>1</samples>
+                <resolution>1</resolution>
+                <min_angle>0.0</min_angle>
+                <max_angle>0.0</max_angle>
+              </vertical>
+            </scan>
+            <range>
+              <min>0.12</min>
+              <max>12.0</max>
+              <resolution>0.01</resolution>
+            </range>
+          </ray>
+          <plugin name="gazebo_ros_gpu_laser" filename="libgazebo_ros_gpu_laser.so">
+            <topicName>/scan</topicName>
+            <frameName>gpu_lidar_link</frameName>
+          </plugin>
+        </sensor>
+      </gazebo>
+    </xacro:unless>
+    <!-- Gazebo Sim GPU lidar (only when using Gazebo Sim) -->
+    <xacro:if value="$(arg use_gz)">
+      <gazebo reference="gpu_lidar_link">
+        <sensor name="gpu_lidar" type="gpu_lidar">
+          <always_on>true</always_on>
+          <update_rate>20</update_rate>
+          <visualize>true</visualize>
+          <topic>/scan</topic>
+          <!-- SDF for GPU lidar uses a <lidar> block; ensure near clip > 0 -->
+          <lidar>
+            <scan>
+              <horizontal>
+                <samples>720</samples>
+                <resolution>1</resolution>
+                <min_angle>-3.14159</min_angle>
+                <max_angle>3.14159</max_angle>
+              </horizontal>
+              <vertical>
+                <samples>1</samples>
+                <resolution>1</resolution>
+                <min_angle>0.0</min_angle>
+                <max_angle>0.0</max_angle>
+              </vertical>
+            </scan>
+            <range>
+              <min>0.12</min>
+              <max>12.0</max>
+              <resolution>0.01</resolution>
+            </range>
+          </lidar>
+          <!-- Explicit clip distances for GPU-based sensor rendering -->
+          <camera>
+            <clip>
+              <near>0.01</near>
+              <far>100.0</far>
+            </clip>
+          </camera>
+        </sensor>
+      </gazebo>
+    </xacro:if>
   </xacro:macro>
 </robot>

File: slam_bot/src/slambot_description/urdf/slambot.xacro (robot description, xacro)
@@ -1,8 +1,6 @@
 <?xml version="1.0"?>
 <robot xmlns:xacro="http://www.ros.org/wiki/xacro" name="slambot">
-  <!-- Simulation flavor: true = Gazebo Sim (Ignition) via gz_ros2_control, false = Gazebo Classic -->
+  <!-- Simulation flavor: true = Gazebo Sim (Ignition), false = Gazebo Classic -->
   <xacro:arg name="use_gz" default="true"/>
-  <!-- If true in Gazebo Sim, move base kinematically from /cmd_vel (disables wheel physics effect) -->
-  <xacro:arg name="kinematic" default="true"/>
   <!-- Main robot macro so other files (e.g., .urdf wrapper) can include/instantiate -->
   <xacro:macro name="slambot" params="">
@@ -66,85 +64,35 @@
     <xacro:include filename="$(find slambot_description)/urdf/slambot-wheels.xacro" />
     <xacro:slambot_wheels />
-    <!-- Transmissions split out for clarity -->
-    <xacro:include filename="$(find slambot_description)/urdf/slambot-transmissions.xacro" />
-    <xacro:slambot_transmissions />
-    <!-- ros2_control interfaces; hardware plugin varies by sim flavor -->
-    <ros2_control name="slambot_system" type="system">
-      <xacro:if value="$(arg use_gz)">
-        <hardware>
-          <plugin>gz_ros2_control/GazeboSimSystem</plugin>
-        </hardware>
-      </xacro:if>
-      <xacro:unless value="$(arg use_gz)">
-        <hardware>
-          <plugin>gazebo_ros2_control/GazeboSystem</plugin>
-        </hardware>
-      </xacro:unless>
-      <joint name="front_left_wheel_joint">
-        <command_interface name="velocity"/>
-        <state_interface name="position"/>
-        <state_interface name="velocity"/>
-      </joint>
-      <joint name="front_right_wheel_joint">
-        <command_interface name="velocity"/>
-        <state_interface name="position"/>
-        <state_interface name="velocity"/>
-      </joint>
-      <joint name="back_left_wheel_joint">
-        <command_interface name="velocity"/>
-        <state_interface name="position"/>
-        <state_interface name="velocity"/>
-      </joint>
-      <joint name="back_right_wheel_joint">
-        <command_interface name="velocity"/>
-        <state_interface name="position"/>
-        <state_interface name="velocity"/>
-      </joint>
-    </ros2_control>
+    <!-- Transmissions are not needed when using kinematic base only; omit ros2_control. -->
+    <!-- ros2_control removed; always use kinematic base in simulation. -->
     <xacro:if value="$(arg use_gz)">
       <gazebo>
-        <plugin
-            name="gz_ros2_control::GazeboSimROS2ControlPlugin"
-            filename="libgz_ros2_control-system.so">
-          <ros2_control>
-            slambot_system
-          </ros2_control>
-          <parameters>$(find slambot_description)/config/mecanum_controller.yaml</parameters>
+        <!-- Always use custom kinematic base plugin in Gazebo Sim -->
+        <plugin name="slambot_kinematic_base" filename="libslambot_kinematic_base.so">
+          <topic>/cmd_vel</topic>
+          <max_linear>1.5</max_linear>
+          <max_angular>3.0</max_angular>
+          <publish_rate>50.0</publish_rate>
+          <publish_odom>false</publish_odom>
+          <odom_topic>/odom</odom_topic>
+          <odom_frame>odom</odom_frame>
+          <base_frame>base_link</base_frame>
+          <pose_cov_diag>0.0001 0.0001 1000000 1000000 1000000 0.001</pose_cov_diag>
+          <twist_cov_diag>0.001 0.001 1000000 1000000 1000000 0.01</twist_cov_diag>
+          <publish_encoders>true</publish_encoders>
+          <ticks_topic>/wheel_encoders</ticks_topic>
+          <joint_state_topic>/encoder_joint_states</joint_state_topic>
+          <ticks_per_rev>2882</ticks_per_rev>
+          <wheel_radius>${wheel_radius}</wheel_radius>
+          <!-- IMPORTANT: These now match your IRL tuned values -->
+          <base_length>${base_length}</base_length>
+          <base_width>${base_width}</base_width>
+          <front_left_joint>front_left_wheel_joint</front_left_joint>
+          <front_right_joint>front_right_wheel_joint</front_right_joint>
+          <back_left_joint>back_left_wheel_joint</back_left_joint>
+          <back_right_joint>back_right_wheel_joint</back_right_joint>
         </plugin>
-        <xacro:if value="$(arg kinematic)">
-          <plugin name="slambot_kinematic_base" filename="libslambot_kinematic_base.so">
-            <topic>/cmd_vel</topic>
-            <max_linear>1.5</max_linear>
-            <max_angular>3.0</max_angular>
-            <publish_rate>50.0</publish_rate>
-            <publish_odom>true</publish_odom>
-            <odom_topic>/odom</odom_topic>
-            <odom_frame>odom</odom_frame>
-            <base_frame>base_link</base_frame>
-            <pose_cov_diag>0.0001 0.0001 1000000 1000000 1000000 0.001</pose_cov_diag>
-            <twist_cov_diag>0.001 0.001 1000000 1000000 1000000 0.01</twist_cov_diag>
-            <publish_encoders>true</publish_encoders>
-            <ticks_topic>/wheel_encoders</ticks_topic>
-            <joint_state_topic>/encoder_joint_states</joint_state_topic>
-            <ticks_per_rev>2882</ticks_per_rev>
-            <wheel_radius>${wheel_radius}</wheel_radius>
-            <!-- IMPORTANT: These now match your IRL tuned values -->
-            <base_length>${base_length}</base_length>
-            <base_width>${base_width}</base_width>
-            <front_left_joint>front_left_wheel_joint</front_left_joint>
-            <front_right_joint>front_right_wheel_joint</front_right_joint>
-            <back_left_joint>back_left_wheel_joint</back_left_joint>
-            <back_right_joint>back_right_wheel_joint</back_right_joint>
-          </plugin>
-        </xacro:if>
       </gazebo>
     </xacro:if>
-    <xacro:unless value="$(arg use_gz)">
-      <gazebo>
-        <plugin name="gazebo_ros2_control" filename="libgazebo_ros2_control.so">
-          <parameters>$(find slambot_description)/config/mecanum_controller.yaml</parameters>
-        </plugin>
-      </gazebo>
-    </xacro:unless>
   </xacro:macro>
   <!-- Instantiate macro by default so this file remains directly usable with xacro -->

Commit message: added slam toolbox (dosent work yet) and changed lidar in urdf to match real life

File: slam_bot/src/slambot_description/urdf/slambot-sensors.xacro (robot description, xacro)
@@ -146,5 +146,5 @@
     </joint>
     <!-- Lidar body/link mounted on top of the plate -->
-    <link name="gpu_lidar_link">
+    <link name="base_laser">
       <inertial>
         <origin xyz="0 0 0" rpy="0 0 0"/>
@@ -169,13 +169,14 @@
       </collision>
     </link>
-    <joint name="gpu_lidar_mount" type="fixed">
+    <joint name="base_laser_mount" type="fixed">
       <parent link="lidar_plate_link"/>
-      <child link="gpu_lidar_link"/>
-      <!-- Sit the lidar on plate top: z = plate half-thickness + lidar half-length = 0.0015 + 0.0125 -->
-      <origin xyz="0 0 0.014" rpy="0 0 0"/>
+      <child link="base_laser"/>
+      <!-- Sit the lidar on plate top: z = plate half-thickness + lidar half-length = 0.0015 + 0.0125
+           Rotate 90 degrees clockwise about +Z (yaw = -pi/2) so sensor arrow points right -->
+      <origin xyz="0 0 0.014" rpy="0 0 -1.57079632679"/>
     </joint>
     <!-- Gazebo Classic GPU lidar (only when NOT using Gazebo Sim) -->
     <xacro:unless value="$(arg use_gz)">
-      <gazebo reference="gpu_lidar_link">
+      <gazebo reference="base_laser">
         <sensor name="gpu_lidar" type="gpu_ray">
           <always_on>1</always_on>
@@ -205,5 +206,5 @@
           <plugin name="gazebo_ros_gpu_laser" filename="libgazebo_ros_gpu_laser.so">
             <topicName>/scan</topicName>
-            <frameName>gpu_lidar_link</frameName>
+            <frameName>base_laser</frameName>
           </plugin>
         </sensor>
@@ -212,5 +213,5 @@
     <!-- Gazebo Sim GPU lidar (only when using Gazebo Sim) -->
     <xacro:if value="$(arg use_gz)">
-      <gazebo reference="gpu_lidar_link">
+      <gazebo reference="base_laser">
         <sensor name="gpu_lidar" type="gpu_lidar">
           <always_on>true</always_on>
